File: HW-10pin/Needle.kicad_pcb (KiCad board)
At the start: 2 copper layers, 24 x 51.8 mm, 14 parts

Commit message: routing
Parts:
- moved REF** 10.4 mm to (131.9, 50.1), turned to 90 degrees
Routing:
- net (no net): track 0.00 -> 510.6 mm
Other:
- board text added: "#RESET"
- board text added: "5V"
- board text added: "GND"
- board text added: "RTCK"
- board text added: "SWCLK/TCK"
- board text added: "SWDIO/TMS"
- board text added: "SWO/TDO"
- board text added: "TDI"
- board text added: "TRST"
- board text added: "Vref"
- board text added: "https://github.com/even-notodd/JTAG_Needle"
